File: PSU_Front_End/PSU_Front_End.kicad_pcb (KiCad board)
At the start: 2 copper layers, 125 x 130 mm, 75 parts, among them J1 ICSP, J10 Banana Plug, J11 Banana Plug, J12 Banana Plug, J13 Banana Plug, J2 ATX Connector, J3 +12V Conn, J4 Banana Plug, J5 Banana Plug, J6 Banana Plug, J7 Banana Plug, J8 Banana Plug, J9 Banana Plug, Q1 2N7002, SW1 Rot Encoder, U1 PIC16F15254-I_SO, U2 MCP45HV51-ST, U3 TPS565242, U4 TMCS1108A2, U5 TMCS1108A2, U6 TMCS1108A2, U7 TMCS1108A2, U8 TMCS1108A2

Commit message: Finished Board Layout
Parts:
- added R10: 10k, Resistor_SMD:R_0805_2012Metric_Pad1.20x1.40mm_HandSolder, B.Cu at (157.5, 62.0)
- added R9: 10k, Resistor_SMD:R_0805_2012Metric_Pad1.20x1.40mm_HandSolder, B.Cu at (157.5, 71.5)
- added SW2: DPDT, psu_front_end:SW DPDT, F.Cu at (137.8, 95.5)
- C1, C16, C18, C19, C2, C24, C3, C4, C5, C6, C7, C8, J1, JP1, L1, Q1, R2, R3, R4, R5, R6, R7, R8, RV1, U2, U3, U8: moved to B.Cu
- R14: renamed from R12; moved to B.Cu
- R21: renamed from R19; moved to B.Cu
- R22: renamed from R20; moved to B.Cu
- U1: footprint footprints:SOIC28_SO_MCH -> Package_SO:SOIC-28W_7.5x18.7mm_P1.27mm; moved to B.Cu
- moved C13 199.7 mm to (197.0, 108.3)
- moved R17 196.8 mm to (180.0, 123.7), turned to -90 degrees
- moved R18 172.0 mm to (160.0, 123.7), turned to -90 degrees
- moved R19 169.0 mm to (140.0, 123.7), turned to -90 degrees
- moved R20 158.5 mm to (120.0, 123.7), turned to -90 degrees
- moved C10 157.9 mm to (154.2, 105.5), turned to 180 degrees
- moved U5 151.9 mm to (160.0, 112.0), turned to 90 degrees
- moved U6 146.8 mm to (140.0, 112.0), turned to 90 degrees
- moved C14 146.3 mm to (154.2, 107.8), turned to 180 degrees
- moved Q1 141.7 mm to (140.0, 83.5), turned to -90 degrees
- moved U4 139.4 mm to (180.0, 112.0), turned to 90 degrees
- moved C1 138.6 mm to (178.5, 71.5), turned to -90 degrees
- moved C9 135.9 mm to (197.0, 110.6)
- moved C17 131.8 mm to (129.5, 109.0), turned to 90 degrees
- moved C21 130.1 mm to (153.2, 111.2), turned to 90 degrees
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- renumbered R9 to R11, R10 to R12, R11 to R13, R13 to R15, R14 to R16, R15 to R17, R16 to R18, R17 to R19, R18 to R20
Connections:
- U4 pad 1: +3V3 -> Net-(J4-Pad1)
- U4 pad 2: +3V3 -> Net-(J4-Pad1)
- U4 pad 3: Net-(J4-Pad1) -> +3V3
- U4 pad 4: Net-(J4-Pad1) -> +3V3
- U5 pad 1: +5V -> Net-(J6-Pad1)
- U5 pad 2: +5V -> Net-(J6-Pad1)
- U5 pad 3: Net-(J6-Pad1) -> +5V
- U5 pad 4: Net-(J6-Pad1) -> +5V
- U6 pad 1: +12V -> Net-(J8-Pad1)
- U6 pad 2: +12V -> Net-(J8-Pad1)
- U6 pad 3: Net-(J8-Pad1) -> +12V
- U6 pad 4: Net-(J8-Pad1) -> +12V
- U7 pad 1: -12V -> Net-(J10-Pad1)
- U7 pad 2: -12V -> Net-(J10-Pad1)
- U7 pad 3: Net-(J10-Pad1) -> -12V
- U7 pad 4: Net-(J10-Pad1) -> -12V
- U8 pad 1: Net-(C16-Pad1) -> Net-(J12-Pad1)
- U8 pad 2: Net-(C16-Pad1) -> Net-(J12-Pad1)
- U8 pad 3: Net-(J12-Pad1) -> Net-(C16-Pad1)
- U8 pad 4: Net-(J12-Pad1) -> Net-(C16-Pad1)
Routing:
- net +12VA: track 0.00 -> 153.0 mm, vias 0 -> 4
- net -12V: track 0.00 -> 129.1 mm, vias 0 -> 1
- net /ENC_{A}: track 0.00 -> 120.0 mm, vias 0 -> 3
- net /ENC_{B}: track 0.00 -> 119.5 mm, vias 0 -> 3
- net /PWR_{OK}: track 0.00 -> 94.4 mm, vias 0 -> 3
- net +3V3: track 0.00 -> 84.1 mm
- net Net-(J12-Pad1): track 0.00 -> 83.6 mm, vias 0 -> 2
- net GND: track 0.00 -> 81.9 mm, vias 0 -> 37
- net /SDA: track 0.00 -> 74.1 mm, vias 0 -> 4
- net /SCL: track 0.00 -> 73.5 mm, vias 0 -> 2
- net /CURR_{+3.3V}: track 0.00 -> 73.2 mm, vias 0 -> 1
- net /~{PS_{ON}}: track 0.00 -> 70.9 mm, vias 0 -> 2
- net Net-(C16-Pad1): track 0.00 -> 56.8 mm, vias 0 -> 3
- net VCC: track 0.00 -> 56.3 mm, vias 0 -> 12
- net /CURR_{-12V}: track 0.00 -> 55.7 mm, vias 0 -> 1
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- added copper zone on F.Cu, net +12V
- added copper zone on F.Cu, net +3V3
- added copper zone on F.Cu, net +5V
- added copper zone on F.Cu, net -12V
- added copper zone on B.Cu, net GND
- added copper zone on F.Cu, net GND
- added copper zone on In1.Cu, net GND
- added copper zone on B.Cu, net Net-(C16-Pad1)
- added copper zone on F.Cu, net Net-(J10-Pad1)
- added copper zone on B.Cu, net Net-(J12-Pad1)
- added copper zone on F.Cu, net Net-(J4-Pad1)
- added copper zone on F.Cu, net Net-(J6-Pad1)
- added copper zone on F.Cu, net Net-(J8-Pad1)
- added copper zone on B.Cu, net Net-(L1-Pad1)
- added copper zone on In2.Cu, net VCC
Other:
- board size 125 x 130 mm -> 100 x 100 mm
- copper layers 2 -> 4
