File: PSU_Front_End/PSU_Front_End.kicad_sch (KiCad schematic)
At the start: 76 parts, among them J1 ICSP, J10 Banana Plug, J11 Banana Plug, J12 Banana Plug, J13 Banana Plug, J2 ATX Connector, J3 +12V Conn, J4 Banana Plug, J5 Banana Plug, J6 Banana Plug, J7 Banana Plug, J8 Banana Plug, J9 Banana Plug, Q1 2N7002, SW1 Rot Encoder, SW2 DPDT, U1 PIC16F15254-I_SO, U2 MCP45HV51-ST, U3 TPS565242, U4 TMCS1108A2, U5 TMCS1108A2, U6 TMCS1108A2, U7 TMCS1108A2, U8 TMCS1108A2

Commit message: Finished Board Layout
Parts:
- added R10, R9: 10k, Resistor_SMD:R_0805_2012Metric_Pad1.20x1.40mm_HandSolder, symbol Device:R_Small
- SW2: footprint (none) -> psu_front_end:SW DPDT
- U1: footprint SOIC28_SO_MCH -> Package_SO:SOIC-28W_7.5x18.7mm_P1.27mm
- renumbered R9 to R11, R10 to R12, R11 to R13, R12 to R14, R13 to R15, R14 to R16, R15 to R17, R16 to R18, R17 to R19, R18 to R20, R19 to R21, R20 to R22
Connections:
- net +12V: now also U6.3 (IN_{-}), U6.4 (IN_{-}); no longer U6.1 (IN_{+}), U6.2 (IN_{+})
- net +3V3: now also U4.3 (IN_{-}), U4.4 (IN_{-}); no longer U4.1 (IN_{+}), U4.2 (IN_{+})
- net +5V: now also U5.3 (IN_{-}), U5.4 (IN_{-}); no longer U5.1 (IN_{+}), U5.2 (IN_{+})
- net -12V: now also U7.3 (IN_{-}), U7.4 (IN_{-}); no longer U7.1 (IN_{+}), U7.2 (IN_{+})
- net SCL: now also R10.2
- net SDA: now also R9.2
- net VCC: now also R10.1, R9.1
- net at J12.1 (Pin_1), R21.1: now also U8.1 (IN_{+}), U8.2 (IN_{+}); no longer U8.3 (IN_{-}), U8.4 (IN_{-})
- net at C16.1, C18.1, C19.1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: now also U8.3 (IN_{-}), U8.4 (IN_{-}); no longer U8.1 (IN_{+}), U8.2 (IN_{+})
- new net: J4.1 (Pin_1), U4.1 (IN_{+}), U4.2 (IN_{+})
- new net: J8.1 (Pin_1), U6.1 (IN_{+}), U6.2 (IN_{+})
- new net: J10.1 (Pin_1), U7.1 (IN_{+}), U7.2 (IN_{+})
- new net: J6.1 (Pin_1), U5.1 (IN_{+}), U5.2 (IN_{+})
Other:
- moved on the sheet: C20, C21, C22, C23, C24, DS1, R2, R3, R4, R5, RV1
